File: hardware/RPi_shield/RPi_shield.kicad_pcb (KiCad board)
At the start: 2 copper layers, 64 x 56.1 mm, 6 parts, among them J1 AudioJack3, J2 AudioJack3, J3 AudioJack3, J4 AudioJack3, J5 RASPBERRY_PI_4B_+_Samtec_ESP-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, M1 Fan

Commit message: add last saves to kicad
Changed lines of the file:
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@@
     (descr "RASPBERRY PI 4B/4GB")
     (tags Connector)
-    (fp_text reference J5 (at -61.440001 -1.518001) (layer F.SilkS)
+    (fp_text reference J5 (at -46.99 3.556) (layer F.SilkS)
       (effects (font (size 1.27 1.27) (thickness 0.254)))
     )
