File: hardware/RPi_shield/RPi_shield.sch (KiCad schematic (older format))
At the start: 6 parts

Commit message: save and push work
Parts:
- J1: renamed from J?; footprint (none) -> digikey-footprints:Phone_Jack_87180-062LF
- J5: renamed from J?; footprint (none) -> Module:Raspberry_Pi_Zero_Socketed_THT_FaceDown_MountingHoles
- M1: renamed from M?; footprint (none) -> Connector_JST:JST_XH_B2B-XH-AM_1x02_P2.50mm_Vertical
- gave numbers to parts that had none: 3
Changed lines of the file:
@@
 $EndDescr
 $Comp
-L Connector:AudioJack2 J?
+L Connector:AudioJack2 J4
 U 1 1 61BCA819
 P 3850 1550
-F 0 "J?" H 3882 1875 50  0000 C CNN
+F 0 "J4" H 3882 1875 50  0000 C CNN
 F 1 "AudioJack2" H 3882 1784 50  0000 C CNN
 F 2 "" H 3850 1550 50  0001 C CNN
@@
 $EndComp
 $Comp
-L power:GND #PWR?
+L power:GND #PWR04
 U 1 1 61BCAB95
 P 4200 1400
-F 0 "#PWR?" H 4200 1150 50  0001 C CNN
+F 0 "#PWR04" H 4200 1150 50  0001 C CNN
 F 1 "GND" H 4205 1227 50  0000 C CNN
 F 2 "" H 4200 1400 50  0001 C CNN
@@
 	4200 1450 4200 1400
 $Comp
-L Connector:Raspberry_Pi_2_3 J?
+L Connector:Raspberry_Pi_2_3 J5
 U 1 1 61BCBBDC
 P 6050 2550
-F 0 "J?" H 6050 4031 50  0000 C CNN
+F 0 "J5" H 6050 4031 50  0000 C CNN
 F 1 "Raspberry_Pi_2_3" H 6050 3940 50  0000 C CNN
-F 2 "" H 6050 2550 50  0001 C CNN
+F 2 "Module:Raspberry_Pi_Zero_Socketed_THT_FaceDown_MountingHoles" H 6050 2550 50  0001 C CNN
 F 3 "https://www.raspberrypi.org/documentation/hardware/raspberrypi/schematics/rpi_SCH_3bplus_1p0_reduced.pdf" H 6050 2550 50  0001 C CNN
 	1    6050 2550
@@
 $EndComp
 $Comp
-L power:GND #PWR?
+L power:GND #PWR06
 U 1 1 61BD036E
 P 6000 4000
-F 0 "#PWR?" H 6000 3750 50  0001 C CNN
+F 0 "#PWR06" H 6000 3750 50  0001 C CNN
 F 1 "GND" H 6005 3827 50  0000 C CNN
 F 2 "" H 6000 4000 50  0001 C CNN
@@
 	6000 3900 6050 3900
 $Comp
-L power:+5V #PWR?
+L power:+5V #PWR05
 U 1 1 61BD1E7D
 P 5850 1100
-F 0 "#PWR?" H 5850 950 50  0001 C CNN
+F 0 "#PWR05" H 5850 950 50  0001 C CNN
 F 1 "+5V" H 5865 1273 50  0000 C CNN
 F 2 "" H 5850 1100 50  0001 C CNN
@@
 	5850 1200 5850 1250
 $Comp
-L Motor:Fan M?
+L Motor:Fan M1
 U 1 1 61BD2C88
 P 8000 1950
-F 0 "M?" H 8158 2046 50  0000 L CNN
+F 0 "M1" H 8158 2046 50  0000 L CNN
 F 1 "Fan" H 8158 1955 50  0000 L CNN
-F 2 "" H 8000 1960 50  0001 C CNN
+F 2 "Connector_JST:JST_XH_B2B-XH-AM_1x02_P2.50mm_Vertical" H 8000 1960 50  0001 C CNN
 F 3 "~" H 8000 1960 50  0001 C CNN
 	1    8000 1950
@@
 $EndComp
 $Comp
-L power:GND #PWR?
+L power:GND #PWR08
 U 1 1 61BD3423
 P 8000 2250
-F 0 "#PWR?" H 8000 2000 50  0001 C CNN
+F 0 "#PWR08" H 8000 2000 50  0001 C CNN
 F 1 "GND" H 8005 2077 50  0000 C CNN
 F 2 "" H 8000 2250 50  0001 C CNN
@@
 	8000 2150 8000 2250
 $Comp
-L power:+5V #PWR?
+L power:+5V #PWR07
 U 1 1 61BD3B74
 P 8000 1500
-F 0 "#PWR?" H 8000 1350 50  0001 C CNN
+F 0 "#PWR07" H 8000 1350 50  0001 C CNN
 F 1 "+5V" H 8015 1673 50  0000 C CNN
 F 2 "" H 8000 1500 50  0001 C CNN
@@
 	4150 1550 4050 1550
 $Comp
-L Connector:AudioJack2 J?
+L Connector:AudioJack2 J3
 U 1 1 61BD70C0
 P 3800 2650
-F 0 "J?" H 3832 2975 50  0000 C CNN
+F 0 "J3" H 3832 2975 50  0000 C CNN
 F 1 "AudioJack2" H 3832 2884 50  0000 C CNN
 F 2 "" H 3800 2650 50  0001 C CNN
@@
 $EndComp
 $Comp
-L power:GND #PWR?
+L power:GND #PWR03
 U 1 1 61BD70C6
 P 4150 2500
-F 0 "#PWR?" H 4150 2250 50  0001 C CNN
+F 0 "#PWR03" H 4150 2250 50  0001 C CNN
 F 1 "GND" H 4155 2327 50  0000 C CNN
 F 2 "" H 4150 2500 50  0001 C CNN
@@
 	4100 2650 4000 2650
 $Comp
-L Connector:AudioJack2 J?
+L Connector:AudioJack2 J2
 U 1 1 61BD7B59
 P 3750 3600
-F 0 "J?" H 3782 3925 50  0000 C CNN
+F 0 "J2" H 3782 3925 50  0000 C CNN
 F 1 "AudioJack2" H 3782 3834 50  0000 C CNN
 F 2 "" H 3750 3600 50  0001 C CNN
@@
 $EndComp
 $Comp
-L power:GND #PWR?
+L power:GND #PWR02
 U 1 1 61BD7B5F
 P 4100 3450
-F 0 "#PWR?" H 4100 3200 50  0001 C CNN
+F 0 "#PWR02" H 4100 3200 50  0001 C CNN
 F 1 "GND" H 4105 3277 50  0000 C CNN
 F 2 "" H 4100 3450 50  0001 C CNN
@@
 	4050 3600 3950 3600
 $Comp
-L Connector:AudioJack2 J?
+L Connector:AudioJack2 J1
 U 1 1 61BD85B7
 P 3700 4450
-F 0 "J?" H 3732 4775 50  0000 C CNN
+F 0 "J1" H 3732 4775 50  0000 C CNN
 F 1 "AudioJack2" H 3732 4684 50  0000 C CNN
-F 2 "" H 3700 4450 50  0001 C CNN
+F 2 "digikey-footprints:Phone_Jack_87180-062LF" H 3700 4450 50  0001 C CNN
 F 3 "~" H 3700 4450 50  0001 C CNN
 	1    3700 4450
@@
 $EndComp
 $Comp
-L power:GND #PWR?
+L power:GND #PWR01
 U 1 1 61BD85BD
 P 4050 4300
-F 0 "#PWR?" H 4050 4050 50  0001 C CNN
+F 0 "#PWR01" H 4050 4050 50  0001 C CNN
 F 1 "GND" H 4055 4127 50  0000 C CNN
 F 2 "" H 4050 4300 50  0001 C CNN

Commit message: finish first iteration of the board and prepare it for kitspace
Parts:
- removed J5: Raspberry_Pi_2_3, Module:Raspberry_Pi_Zero_Socketed_THT_FaceDown_MountingHoles, symbol Connector:Raspberry_Pi_2_3
- added J5: RASPBERRY_PI_4B_+_Samtec_ESP-120-33-G-D, RASPBERRYPI4B4GB, symbol raspberryPi:RASPBERRY_PI_4B_+_Samtec_ESP-120-33-G-D
- added J? (x4): Conn_Coaxial, symbol Connector:Conn_Coaxial
Connections:
- net +5V: now also J5.2 (5V_1), J5.4 (5V_2)
- net GND: now also J5.14 (GND_3), J5.20 (GND_4), J5.25 (GND_5), J5.30 (GND_6), J5.34 (GND_7), J5.39 (GND_8), J5.6 (GND_1), J5.9 (GND_2)
- net jack1: now also J5.28 (BCM_1)
- net jack2: now also J5.29 (BCM_5)
- net jack3: now also J5.21 (BCM_9)
- net jack4: now also J5.33 (BCM_13)

Commit message: add last saves to kicad
Parts:
- removed J1: AudioJack2, digikey-footprints:Phone_Jack_87180-062LF, symbol Connector:AudioJack2
- removed J2, J3, J4: AudioJack2, symbol Connector:AudioJack2
- removed J? (x4): Conn_Coaxial, symbol Connector:Conn_Coaxial
- added J1, J2, J3, J4: AudioJack3, Connector_Audio:Jack_3.5mm_CUI_SJ1-3533NG_Horizontal, symbol Connector:AudioJack3
- J5: footprint RASPBERRYPI4B4GB -> raspberrypi:RASPBERRYPI4B4GB
- M1: footprint Connector_JST:JST_XH_B2B-XH-AM_1x02_P2.50mm_Vertical -> Connector_PinHeader_2.54mm:PinHeader_1x02_P2.54mm_Horizontal
Connections:
- net GND: now also J1.S, J2.S, J3.S, J4.S
- net jack1: now also J3.R, J3.T
- net jack2: now also J2.R, J2.T
- net jack3: now also J1.R, J1.T
- net jack4: now also J4.R, J4.T
Changed lines of the file:
@@
 $EndDescr
-$Comp
-L Connector:AudioJack2 J4
-U 1 1 61BCA819
-P 3850 1550
-F 0 "J4" H 3882 1875 50  0000 C CNN
-F 1 "AudioJack2" H 3882 1784 50  0000 C CNN
-F 2 "" H 3850 1550 50  0001 C CNN
-F 3 "~" H 3850 1550 50  0001 C CNN
-	1    3850 1550
-	1    0    0    -1
-$EndComp
 $Comp
 L power:GND #PWR04
@@
 F 0 "M1" H 8158 2046 50  0000 L CNN
 F 1 "Fan" H 8158 1955 50  0000 L CNN
-F 2 "Connector_JST:JST_XH_B2B-XH-AM_1x02_P2.50mm_Vertical" H 8000 1960 50  0001 C CNN
+F 2 "Connector_PinHeader_2.54mm:PinHeader_1x02_P2.54mm_Horizontal" H 8000 1960 50  0001 C CNN
 F 3 "~" H 8000 1960 50  0001 C CNN
 	1    8000 1950
@@
 jack1
 Wire Wire Line
-	4150 1550 4050 1550
-$Comp
-L Connector:AudioJack2 J3
-U 1 1 61BD70C0
-P 3800 2650
-F 0 "J3" H 3832 2975 50  0000 C CNN
-F 1 "AudioJack2" H 3832 2884 50  0000 C CNN
-F 2 "" H 3800 2650 50  0001 C CNN
-F 3 "~" H 3800 2650 50  0001 C CNN
-	1    3800 2650
-	1    0    0    -1
-$EndComp
+	4150 1550 4100 1550
 $Comp
 L power:GND #PWR03
@@
 jack2
 Wire Wire Line
-	4100 2650 4000 2650
-$Comp
-L Connector:AudioJack2 J2
-U 1 1 61BD7B59
-P 3750 3600
-F 0 "J2" H 3782 3925 50  0000 C CNN
-F 1 "AudioJack2" H 3782 3834 50  0000 C CNN
-F 2 "" H 3750 3600 50  0001 C CNN
-F 3 "~" H 3750 3600 50  0001 C CNN
-	1    3750 3600
-	1    0    0    -1
-$EndComp
+	4100 2650 4050 2650
 $Comp
 L power:GND #PWR02
@@
 jack3
 Wire Wire Line
-	4050 3600 3950 3600
-$Comp
-L Connector:AudioJack2 J1
-U 1 1 61BD85B7
-P 3700 4450
-F 0 "J1" H 3732 4775 50  0000 C CNN
-F 1 "AudioJack2" H 3732 4684 50  0000 C CNN
-F 2 "digikey-footprints:Phone_Jack_87180-062LF" H 3700 4450 50  0001 C CNN
-F 3 "~" H 3700 4450 50  0001 C CNN
-	1    3700 4450
-	1    0    0    -1
-$EndComp
+	4050 3600 4000 3600
 $Comp
 L power:GND #PWR01
@@
 jack4
 Wire Wire Line
-	4000 4450 3900 4450
+	4000 4450 3950 4450
 $Comp
 L raspberryPi:RASPBERRY_PI_4B_+_Samtec_ESP-120-33-G-D J5
@@
 F 0 "J5" H 6250 4615 50  0000 C CNN
 F 1 "RASPBERRY_PI_4B_+_Samtec_ESP-120-33-G-D" H 6250 4524 50  0000 C CNN
-F 2 "RASPBERRYPI4B4GB" H 6750 4450 50  0001 L CNN
+F 2 "raspberrypi:RASPBERRYPI4B4GB" H 6750 4450 50  0001 L CNN
 F 3 "https://www.raspberrypi.org/documentation/hardware/raspberrypi/mechanical/rpi_MECH_4b_4p0.pdf" H 6750 4350 50  0001 L CNN
 F 4 "RASPBERRY PI 4 MODEL B with Samtec ESP-120-33-G-D connector drawn from underneath for use as a plug in module." H 6750 4250 50  0001 L CNN "Description"
@@
 NoConn ~ 5600 4450
 $Comp
-L Connector:Conn_Coaxial J?
-U 1 1 61C488EE
-P 4700 1450
-F 0 "J?" H 4800 1425 50  0000 L CNN
-F 1 "Conn_Coaxial" H 4800 1334 50  0000 L CNN
-F 2 "" H 4700 1450 50  0001 C CNN
-F 3 " ~" H 4700 1450 50  0001 C CNN
-	1    4700 1450
-	1    0    0    -1
-$EndComp
-$Comp
-L Connector:Conn_Coaxial J?
-U 1 1 61C496EC
-P 4650 2550
-F 0 "J?" H 4750 2525 50  0000 L CNN
-F 1 "Conn_Coaxial" H 4750 2434 50  0000 L CNN
-F 2 "" H 4650 2550 50  0001 C CNN
-F 3 " ~" H 4650 2550 50  0001 C CNN
-	1    4650 2550
-	1    0    0    -1
-$EndComp
-$Comp
-L Connector:Conn_Coaxial J?
-U 1 1 61C49B88
-P 4650 3450
-F 0 "J?" H 4750 3425 50  0000 L CNN
-F 1 "Conn_Coaxial" H 4750 3334 50  0000 L CNN
-F 2 "" H 4650 3450 50  0001 C CNN
-F 3 " ~" H 4650 3450 50  0001 C CNN
-	1    4650 3450
-	1    0    0    -1
-$EndComp
-$Comp
-L Connector:Conn_Coaxial J?
-U 1 1 61C4A228
-P 4650 4350
-F 0 "J?" H 4750 4325 50  0000 L CNN
-F 1 "Conn_Coaxial" H 4750 4234 50  0000 L CNN
-F 2 "" H 4650 4350 50  0001 C CNN
-F 3 " ~" H 4650 4350 50  0001 C CNN
-	1    4650 4350
-	1    0    0    -1
-$EndComp
+L Connector:AudioJack3 J4
+U 1 1 61C4B35F
+P 3700 4450
+F 0 "J4" H 3682 4775 50  0000 C CNN
+F 1 "AudioJack3" H 3682 4684 50  0000 C CNN
+F 2 "Connector_Audio:Jack_3.5mm_CUI_SJ1-3533NG_Horizontal" H 3700 4450 50  0001 C CNN
+F 3 "~" H 3700 4450 50  0001 C CNN
+	1    3700 4450
+	1    0    0    -1
+$EndComp
+Wire Wire Line
+	3950 4450 3950 4550
+Wire Wire Line
+	3950 4550 3900 4550
+Connection ~ 3950 4450
+Wire Wire Line
+	3950 4450 3900 4450
+$Comp
+L Connector:AudioJack3 J1
+U 1 1 61C53EA3
+P 3750 3600
+F 0 "J1" H 3732 3925 50  0000 C CNN
+F 1 "AudioJack3" H 3732 3834 50  0000 C CNN
+F 2 "Connector_Audio:Jack_3.5mm_CUI_SJ1-3533NG_Horizontal" H 3750 3600 50  0001 C CNN
+F 3 "~" H 3750 3600 50  0001 C CNN
+	1    3750 3600
+	1    0    0    -1
+$EndComp
+$Comp
+L Connector:AudioJack3 J2
+U 1 1 61C546DE
+P 3800 2650
+F 0 "J2" H 3782 2975 50  0000 C CNN
+F 1 "AudioJack3" H 3782 2884 50  0000 C CNN
+F 2 "Connector_Audio:Jack_3.5mm_CUI_SJ1-3533NG_Horizontal" H 3800 2650 50  0001 C CNN
+F 3 "~" H 3800 2650 50  0001 C CNN
+	1    3800 2650
+	1    0    0    -1
+$EndComp
+$Comp
+L Connector:AudioJack3 J3
+U 1 1 61C5505F
+P 3850 1550
+F 0 "J3" H 3832 1875 50  0000 C CNN
+F 1 "AudioJack3" H 3832 1784 50  0000 C CNN
+F 2 "Connector_Audio:Jack_3.5mm_CUI_SJ1-3533NG_Horizontal" H 3850 1550 50  0001 C CNN
+F 3 "~" H 3850 1550 50  0001 C CNN
+	1    3850 1550
+	1    0    0    -1
+$EndComp
+Wire Wire Line
+	4100 1550 4100 1650
+Wire Wire Line
+	4100 1650 4050 1650
+Connection ~ 4100 1550
+Wire Wire Line
+	4100 1550 4050 1550
+Wire Wire Line
+	4050 2650 4050 2750
+Wire Wire Line
+	4050 2750 4000 2750
+Connection ~ 4050 2650
+Wire Wire Line
+	4050 2650 4000 2650
+Wire Wire Line
+	4000 3600 4000 3700
+Wire Wire Line
+	4000 3700 3950 3700
+Connection ~ 4000 3600
+Wire Wire Line
+	4000 3600 3950 3600
 $EndSCHEMATC
