File: hardware/RPi_shield/_autosave-RPi_shield.kicad_pcb (KiCad board)
At the start: 2 copper layers, 64 x 56.1 mm, 6 parts, among them J1 AudioJack3, J2 AudioJack3, J3 AudioJack3, J4 AudioJack3, J5 RASPBERRY_PI_4B_+_Samtec_ESP-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, M1 Fan

Commit message: reverse labeling and add logo
Parts:
- added G***: LOGO, board_logo:board_logo, B.Cu at (87.6, 53.8)
